Commit message: fix: change joint limit

File: fairino_description/urdf/fairino20_v6.urdf (robot description, URDF)
Before this commit: robot fairino20_v6_robot, 7 links, 6 joints
Joints:
- joint j1: origin xyz=0 0 0 rpy=0 0 0 -> xyz=0 0 0 rpy=0 0 3.1415

Commit message: fix: v3.7.6

File: fairino_description/urdf/fairino20_v6.urdf (robot description, URDF)
Before this commit: robot fairino20_v6_robot, 7 links, 6 joints
Joints:
- joint j1: origin xyz=0 0 0 rpy=0 0 3.1415 -> xyz=0 0 0 rpy=0 0 0
